File: kicad/Clicky SNES Controller Kicad.sch (KiCad schematic (older format))
At the start: 36 parts, among them CN1 CN1, P11 TL_IN, P13 TR_IN, P2 VSS_Trigger, P3 TR_TL_OUT, P4 DPAD_IN, P6 ABXY_IN, U1 4021, U2 4021, X1 SW_PUSH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

Commit message: change pads on passives to non hand-soldering versions
Parts:
- C1, C2: footprint Capacitors_SMD:C_1206_HandSoldering -> Capacitors_SMD:C_1206
- R1, R10, R11, R12, R13, R14, R15, R16, R17, R18, R2, R7, R8, R9: footprint Resistors_SMD:R_1206_HandSoldering -> Resistors_SMD:R_1206
Changed lines of the file:
@@
 F 0 "R1" V 1330 1450 50  0000 C CNN
 F 1 "47k" V 1250 1450 50  0000 C CNN
-F 2 "Resistors_SMD:R_1206_HandSoldering" V 1180 1450 50  0001 C CNN
+F 2 "Resistors_SMD:R_1206" V 1180 1450 50  0001 C CNN
 F 3 "" H 1250 1450 50  0000 C CNN
 	1    1250 1450
@@
 F 0 "R2" V 1330 1650 50  0000 C CNN
 F 1 "47k" V 1250 1650 50  0000 C CNN
-F 2 "Resistors_SMD:R_1206_HandSoldering" V 1180 1650 50  0001 C CNN
+F 2 "Resistors_SMD:R_1206" V 1180 1650 50  0001 C CNN
 F 3 "" H 1250 1650 50  0000 C CNN
 	1    1250 1650
@@
 F 0 "R7" V 4900 2650 50  0000 C CNN
 F 1 "47k" V 4850 2850 50  0000 C CNN
-F 2 "Resistors_SMD:R_1206_HandSoldering" V 4780 2850 50  0001 C CNN
+F 2 "Resistors_SMD:R_1206" V 4780 2850 50  0001 C CNN
 F 3 "" H 4850 2850 50  0000 C CNN
 	1    4850 2850
@@
 F 0 "R8" V 4900 2750 50  0000 C CNN
 F 1 "47k" V 4850 2950 50  0000 C CNN
-F 2 "Resistors_SMD:R_1206_HandSoldering" V 4780 2950 50  0001 C CNN
+F 2 "Resistors_SMD:R_1206" V 4780 2950 50  0001 C CNN
 F 3 "" H 4850 2950 50  0000 C CNN
 	1    4850 2950
@@
 F 0 "R9" V 4900 2850 50  0000 C CNN
 F 1 "47k" V 4850 3050 50  0000 C CNN
-F 2 "Resistors_SMD:R_1206_HandSoldering" V 4780 3050 50  0001 C CNN
+F 2 "Resistors_SMD:R_1206" V 4780 3050 50  0001 C CNN
 F 3 "" H 4850 3050 50  0000 C CNN
 	1    4850 3050
@@
 F 0 "R10" V 4900 2950 50  0000 C CNN
 F 1 "47k" V 4850 3150 50  0000 C CNN
-F 2 "Resistors_SMD:R_1206_HandSoldering" V 4780 3150 50  0001 C CNN
+F 2 "Resistors_SMD:R_1206" V 4780 3150 50  0001 C CNN
 F 3 "" H 4850 3150 50  0000 C CNN
 	1    4850 3150
@@
 F 0 "R11" V 1600 2200 50  0000 C CNN
 F 1 "47k" V 1550 2450 50  0000 C CNN
-F 2 "Resistors_SMD:R_1206_HandSoldering" V 1480 2450 50  0001 C CNN
+F 2 "Resistors_SMD:R_1206" V 1480 2450 50  0001 C CNN
 F 3 "" H 1550 2450 50  0000 C CNN
 	1    1550 2450
@@
 F 0 "R12" V 1600 2300 50  0000 C CNN
 F 1 "47k" V 1550 2550 50  0000 C CNN
-F 2 "Resistors_SMD:R_1206_HandSoldering" V 1480 2550 50  0001 C CNN
+F 2 "Resistors_SMD:R_1206" V 1480 2550 50  0001 C CNN
 F 3 "" H 1550 2550 50  0000 C CNN
 	1    1550 2550
@@
 F 0 "R13" V 1600 2400 50  0000 C CNN
 F 1 "47k" V 1550 2650 50  0000 C CNN
-F 2 "Resistors_SMD:R_1206_HandSoldering" V 1480 2650 50  0001 C CNN
+F 2 "Resistors_SMD:R_1206" V 1480 2650 50  0001 C CNN
 F 3 "" H 1550 2650 50  0000 C CNN
 	1    1550 2650
@@
 F 0 "R14" V 1600 2500 50  0000 C CNN
 F 1 "47k" V 1550 2750 50  0000 C CNN
-F 2 "Resistors_SMD:R_1206_HandSoldering" V 1480 2750 50  0001 C CNN
+F 2 "Resistors_SMD:R_1206" V 1480 2750 50  0001 C CNN
 F 3 "" H 1550 2750 50  0000 C CNN
 	1    1550 2750
@@
 F 0 "R15" V 1600 2600 50  0000 C CNN
 F 1 "47k" V 1550 2850 50  0000 C CNN
-F 2 "Resistors_SMD:R_1206_HandSoldering" V 1480 2850 50  0001 C CNN
+F 2 "Resistors_SMD:R_1206" V 1480 2850 50  0001 C CNN
 F 3 "" H 1550 2850 50  0000 C CNN
 	1    1550 2850
@@
 F 0 "R16" V 1600 2700 50  0000 C CNN
 F 1 "47k" V 1550 2950 50  0000 C CNN
-F 2 "Resistors_SMD:R_1206_HandSoldering" V 1480 2950 50  0001 C CNN
+F 2 "Resistors_SMD:R_1206" V 1480 2950 50  0001 C CNN
 F 3 "" H 1550 2950 50  0000 C CNN
 	1    1550 2950
@@
 F 0 "R17" V 1600 2800 50  0000 C CNN
 F 1 "47k" V 1550 3050 50  0000 C CNN
-F 2 "Resistors_SMD:R_1206_HandSoldering" V 1480 3050 50  0001 C CNN
+F 2 "Resistors_SMD:R_1206" V 1480 3050 50  0001 C CNN
 F 3 "" H 1550 3050 50  0000 C CNN
 	1    1550 3050
@@
 F 0 "R18" V 1600 2900 50  0000 C CNN
 F 1 "47k" V 1550 3150 50  0000 C CNN
-F 2 "Resistors_SMD:R_1206_HandSoldering" V 1480 3150 50  0001 C CNN
+F 2 "Resistors_SMD:R_1206" V 1480 3150 50  0001 C CNN
 F 3 "" H 1550 3150 50  0000 C CNN
 	1    1550 3150
@@
 F 0 "C1" H 2575 1400 50  0000 L CNN
 F 1 ".1u" H 2700 1300 50  0000 L CNN
-F 2 "Capacitors_SMD:C_1206_HandSoldering" H 2588 1150 50  0001 C CNN
+F 2 "Capacitors_SMD:C_1206" H 2588 1150 50  0001 C CNN
 F 3 "" H 2550 1300 50  0000 C CNN
 F 4 "Place near U1" H 2550 1300 60  0001 C CNN "Note"
@@
 F 0 "C2" H 5875 1400 50  0000 L CNN
 F 1 ".1u" H 6000 1300 50  0000 L CNN
-F 2 "Capacitors_SMD:C_1206_HandSoldering" H 5888 1150 50  0001 C CNN
+F 2 "Capacitors_SMD:C_1206" H 5888 1150 50  0001 C CNN
 F 3 "" H 5850 1300 50  0000 C CNN
 F 4 "Place near U2" H 5850 1300 60  0001 C CNN "Note"
@@
 Connection ~ 5100 6550
 Wire Wire Line
-	5100 6850 5100 6000
+	5100 6000 5100 6850
 Wire Wire Line
 	6350 6250 6350 7200
@@
 	5700 6150 5400 6150
 Wire Wire Line
-	5400 7100 5400 6150
+	5400 6150 5400 7100
 Wire Wire Line
 	2400 6000 2750 6000
@@
 	5050 6400 4650 6400
 Wire Wire Line
-	4650 7050 4650 6400
+	4650 6400 4650 7050
 Wire Wire Line
 	1750 7100 1750 6250
 Connection ~ 3600 7050
 Wire Wire Line
-	3050 7050 4650 7050
+	4650 7050 3050 7050
 Wire Wire Line
 	3600 7050 3600 7250
@@
 	6350 7200 3900 7200
 Wire Wire Line
-	1800 6850 5100 6850
+	5100 6850 1800 6850
 Wire Wire Line
 	2750 6900 3900 6900
@@
 	2400 6950 3800 6950
 Wire Wire Line
-	1750 7100 5400 7100
+	5400 7100 1750 7100
 Text Notes 3500 6800 0    60   ~ 0
 Main Board

Commit message: Route TR/TL through the board-to-board connectors
Having TR and TL connectors on the main board puts them too far
away from the trigger boards. This prevents the existing wires
on those boards from being reused.

Move the connectors to the center of the top edge of the ABXY
and DPAD boards (a single connector can be used on both boards).
This combines P11 and P13 (now P15).

P15 is routed straight to the board-to-board connectors so that
it can be brought onto the main board. This changes these from
1x5 to 1x6 pin headers. I have changed the designator for these:
P4 -> P14
P6 -> P16

I have also changed the board-to-board connectors to 2.54mm
pitch because the 1.27mm pitch was extremely tedious to hand-
solder.
Parts:
- removed P13: TR_IN, Pin_Headers:Pin_Header_Angled_1x02_Pitch2.54mm, symbol CONN_01X02
- CN1: footprint Pin_Headers:Pin_Header_Angled_1x05_Pitch2.54mm -> Extra_Pin_Headers:Pin_Header_Angled_1x05_Pitch2.54mm_Sinister
- P14: renamed from P4; footprint Pin_Headers:Pin_Header_Straight_1x05_Pitch1.27mm -> Pin_Headers:Pin_Header_Straight_1x06_Pitch2.54mm; symbol CONN_01X05 -> CONN_01X06
- P15: renamed from P11; value TL_IN -> TR_TL_IN; footprint Pin_Headers:Pin_Header_Angled_1x02_Pitch2.54mm -> Pin_Headers:Pin_Header_Straight_1x02_Pitch2.54mm
- P16: renamed from P6; footprint Pin_Headers:Pin_Header_Straight_1x05_Pitch1.27mm -> Pin_Headers:Pin_Header_Straight_1x06_Pitch2.54mm; symbol CONN_01X05 -> CONN_01X06
Connections:
- net Right: now also P14.6 (P6); no longer P14.5 (P5)
- net TL: now also P14.5 (P5)
- net TR: now also P16.5 (P5)
- net Y: now also P16.6 (P6); no longer P16.5 (P5)
Other:
- note added: "Wiring Harnesses --\n1. SNES Controller <-> CN1\n2. DPAD_IN (DPAD Board) <-> DPAD_IN (Main Board)\n3. DPAD_IN (ABXY Board) <-> ABXY_IN (Main Board)\n3. TR_TL_IN <-> Trigger Board\n (1) GND -> VSS_Trigger\n (2) TR_TL <- TR_TL_switch\n\n(Unless otherwise noted, pins are connected 1-to-1.)"
- note removed: "Wiring Harnesses --\n1. SNES Controller <-> CN1\n2. DPAD_IN (DPAD Board) <-> DPAD_IN (Main Board)\n3. DPAD_IN (ABXY Board) <-> ABXY_IN (Main Board)\n3. TR_IN <-> Trigger Board\n (1) TR <- TR_TL_switch\n (2) GND -> VSS_Trigger\n4. TL_IN <-> Trigger Board\n (1) TL <- TR_TL_switch\n (2) GND -> VSS_Trigger\n\n(Unless otherwise noted, pins are connected 1-to-1.)"
- moved on the sheet: P15
Changed lines of the file:
@@
 F 0 "CN1" H 1600 1250 50  0000 C CNN
 F 1 "CN1" V 1700 950 50  0000 C CNN
-F 2 "Pin_Headers:Pin_Header_Angled_1x05_Pitch2.54mm" H 1600 950 50  0001 C CNN
+F 2 "Extra_Pin_Headers:Pin_Header_Angled_1x05_Pitch2.54mm_Sinister" H 1600 950 50  0001 C CNN
 F 3 "" H 1600 950 50  0000 C CNN
 	1    1600 950
@@
 Duplicate of Left Trigger
 $Comp
-L CONN_01X02 P13
-U 1 1 58AC1D3C
-P 3600 5700
-F 0 "P13" H 3600 5850 50  0000 C CNN
-F 1 "TR_IN" V 3700 5700 50  0000 C CNN
-F 2 "Pin_Headers:Pin_Header_Angled_1x02_Pitch2.54mm" H 3600 5700 50  0001 C CNN
-F 3 "" H 3600 5700 50  0000 C CNN
-	1    3600 5700
+L CONN_01X02 P15
+U 1 1 58AC1D42
+P 3450 5700
+F 0 "P15" H 3450 5850 50  0000 C CNN
+F 1 "TR_TL_IN" V 3550 5700 50  0000 C CNN
+F 2 "Pin_Headers:Pin_Header_Straight_1x02_Pitch2.54mm" H 3450 5700 50  0001 C CNN
+F 3 "" H 3450 5700 50  0000 C CNN
+	1    3450 5700
 	0    -1   -1   0
 $EndComp
-$Comp
-L CONN_01X02 P11
-U 1 1 58AC1D42
-P 3300 5700
-F 0 "P11" H 3300 5850 50  0000 C CNN
-F 1 "TL_IN" V 3400 5700 50  0000 C CNN
-F 2 "Pin_Headers:Pin_Header_Angled_1x02_Pitch2.54mm" H 3300 5700 50  0001 C CNN
-F 3 "" H 3300 5700 50  0000 C CNN
-	1    3300 5700
-	0    -1   -1   0
-$EndComp
-Text Label 3650 5900 3    60   ~ 0
+Text Label 4200 5900 3    60   ~ 0
 TR
-Text Label 3350 5900 3    60   ~ 0
+Text Label 3600 7250 1    60   ~ 0
 TL
 Text Label 2400 6000 0    60   ~ 0
@@
 VSS_Trigger
 Text Notes 1050 4850 0    60   ~ 0
-Wiring Harnesses --\n1. SNES Controller <-> CN1\n2. DPAD_IN (DPAD Board) <-> DPAD_IN (Main Board)\n3. DPAD_IN (ABXY Board) <-> ABXY_IN (Main Board)\n3. TR_IN <-> Trigger Board\n   (1) TR <- TR_TL_switch\n   (2) GND -> VSS_Trigger\n4. TL_IN <-> Trigger Board\n   (1) TL <- TR_TL_switch\n   (2) GND -> VSS_Trigger\n\n(Unless otherwise noted, pins are connected 1-to-1.)
+Wiring Harnesses --\n1. SNES Controller <-> CN1\n2. DPAD_IN (DPAD Board) <-> DPAD_IN (Main Board)\n3. DPAD_IN (ABXY Board) <-> ABXY_IN (Main Board)\n3. TR_TL_IN <-> Trigger Board\n   (1) GND -> VSS_Trigger\n   (2) TR_TL <- TR_TL_switch\n\n(Unless otherwise noted, pins are connected 1-to-1.)
 $Comp
 L 4021 U1
@@
 L GND #PWR014
 U 1 1 58D7D6A9
-P 3250 5950
-F 0 "#PWR014" H 3250 5700 50  0001 C CNN
-F 1 "GND" H 3250 5800 50  0000 C CNN
-F 2 "" H 3250 5950 50  0000 C CNN
-F 3 "" H 3250 5950 50  0000 C CNN
-	1    3250 5950
+P 3400 5950
+F 0 "#PWR014" H 3400 5700 50  0001 C CNN
+F 1 "GND" H 3400 5800 50  0000 C CNN
+F 2 "" H 3400 5950 50  0000 C CNN
+F 3 "" H 3400 5950 50  0000 C CNN
+	1    3400 5950
 	1    0    0    -1
 $EndComp
@@
 B_switch
 $Comp
+L CONN_01X06 P14
+U 1 1 58D7F440
+P 3750 7450
+F 0 "P14" H 3750 7100 50  0000 C CNN
+F 1 "DPAD_IN" V 3850 7450 50  0000 C CNN
+F 2 "Pin_Headers:Pin_Header_Straight_1x06_Pitch2.54mm" H 3750 7450 50  0001 C CNN
+F 3 "" H 3750 7450 50  0000 C CNN
+	1    3750 7450
+	0    1    1    0
+$EndComp
+$Comp
+L CONN_01X06 P16
+U 1 1 58D7F9B5
+P 4050 5700
+F 0 "P16" H 4050 6050 50  0000 C CNN
+F 1 "ABXY_IN" V 4150 5700 50  0000 C CNN
+F 2 "Pin_Headers:Pin_Header_Straight_1x06_Pitch2.54mm" H 4050 5700 50  0001 C CNN
+F 3 "" H 4050 5700 50  0000 C CNN
+	1    4050 5700
+	0    -1   -1   0
+$EndComp
+$Comp
 L GND #PWR015
-U 1 1 58D7EACD
-P 3550 5950
-F 0 "#PWR015" H 3550 5700 50  0001 C CNN
-F 1 "GND" H 3550 5800 50  0000 C CNN
-F 2 "" H 3550 5950 50  0000 C CNN
-F 3 "" H 3550 5950 50  0000 C CNN
-	1    3550 5950
-	1    0    0    -1
-$EndComp
-$Comp
-L CONN_01X05 P4
-U 1 1 58D7F440
-P 3800 7450
-F 0 "P4" H 3800 7750 50  0000 C CNN
-F 1 "DPAD_IN" V 3900 7450 50  0000 C CNN
-F 2 "Pin_Headers:Pin_Header_Straight_1x05_Pitch1.27mm" H 3800 7450 50  0001 C CNN
-F 3 "" H 3800 7450 50  0000 C CNN
-	1    3800 7450
-	0    1    1    0
-$EndComp
-$Comp
-L CONN_01X05 P6
-U 1 1 58D7F9B5
-P 4100 5700
-F 0 "P6" H 4100 6000 50  0000 C CNN
-F 1 "ABXY_IN" V 4200 5700 50  0000 C CNN
-F 2 "Pin_Headers:Pin_Header_Straight_1x05_Pitch1.27mm" H 4100 5700 50  0001 C CNN
-F 3 "" H 4100 5700 50  0000 C CNN
-	1    4100 5700
-	0    -1   -1   0
-$EndComp
-$Comp
-L GND #PWR016
 U 1 1 58D824DC
-P 3900 5950
-F 0 "#PWR016" H 3900 5700 50  0001 C CNN
-F 1 "GND" H 3900 5800 50  0000 C CNN
-F 2 "" H 3900 5950 50  0000 C CNN
-F 3 "" H 3900 5950 50  0000 C CNN
-	1    3900 5950
+P 3800 5950
+F 0 "#PWR015" H 3800 5700 50  0001 C CNN
+F 1 "GND" H 3800 5800 50  0000 C CNN
+F 2 "" H 3800 5950 50  0000 C CNN
+F 3 "" H 3800 5950 50  0000 C CNN
+	1    3800 5950
 	1    0    0    -1
 $EndComp
@@
 Text Label 3700 7250 1    60   ~ 0
 Left
-Text Label 3600 7250 1    60   ~ 0
+Text Label 3500 7250 1    60   ~ 0
 Right
+Text Label 3900 5900 3    60   ~ 0
+A
 Text Label 4000 5900 3    60   ~ 0
-A
+B
 Text Label 4100 5900 3    60   ~ 0
-B
-Text Label 4200 5900 3    60   ~ 0
 X
 Text Label 4300 5900 3    60   ~ 0
 Y
+$Comp
+L GND #PWR016
+U 1 1 58D85E74
+P 4250 7350
+F 0 "#PWR016" H 4250 7100 50  0001 C CNN
+F 1 "GND" H 4250 7200 50  0000 C CNN
+F 2 "" H 4250 7350 50  0000 C CNN
+F 3 "" H 4250 7350 50  0000 C CNN
+	1    4250 7350
+	1    0    0    -1
+$EndComp
+Text Notes 3500 6800 0    60   ~ 0
+Main Board
+Text Notes 1800 7050 0    60   ~ 0
+DPAD Board
+Text Notes 5150 7050 0    60   ~ 0
+ABXY Board
 Connection ~ 3350 6550
 Wire Wire Line
@@
 	3000 6700 4450 6700
 Wire Wire Line
-	3550 5900 3550 5950
-Wire Wire Line
-	3250 5900 3250 5950
-Wire Wire Line
-	3900 5950 3900 5900
+	3800 5950 3800 5900
 Wire Wire Line
 	5050 6250 5050 6400
@@
 Wire Wire Line
 	1750 7100 1750 6250
-Connection ~ 3600 7050
 Wire Wire Line
 	4650 7050 3050 7050
-Wire Wire Line
-	3600 7050 3600 7250
 Connection ~ 3700 7100
 Connection ~ 3800 7150
@@
 	3900 6900 3900 7250
 Connection ~ 4000 6850
-$Comp
-L GND #PWR017
-U 1 1 58D85E74
-P 4250 7350
-F 0 "#PWR017" H 4250 7100 50  0001 C CNN
-F 1 "GND" H 4250 7200 50  0000 C CNN
-F 2 "" H 4250 7350 50  0000 C CNN
-F 3 "" H 4250 7350 50  0000 C CNN
-	1    4250 7350
-	1    0    0    -1
-$EndComp
 Wire Wire Line
 	4250 7250 4250 7350
@@
 Wire Wire Line
 	5400 7100 1750 7100
-Text Notes 3500 6800 0    60   ~ 0
-Main Board
 Wire Wire Line
 	3350 6600 3350 6550
-Text Notes 1800 7050 0    60   ~ 0
-DPAD Board
-Text Notes 5150 7050 0    60   ~ 0
-ABXY Board
+Wire Wire Line
+	3400 5900 3400 5950
+Text Label 3500 5900 0    60   ~ 0
+TR_TL
+Wire Wire Line
+	3500 7050 3500 7250
+Connection ~ 3500 7050
+Wire Wire Line
+	3600 7250 3600 6650
+Wire Wire Line
+	3600 6650 3500 6650
+Wire Wire Line
+	3500 6650 3500 5900
 $EndSCHEMATC
